File: dcc-adapter-board-kato-1.310-21mtc.kicad_pcb (KiCad board)
At the start: 2 copper layers, 59.5 x 16 mm, 27 parts, among them Q1 NMOSFET1, Q2 NMOSFET2

Commit message: v3
Other:
- board text added: "K 1-310 21MTC Adaptor Board ver. 3 2023.06.15 岡本和樹"
- board text removed: "K 1-310 21MTC Adaptor Board ver. 2 2023.05.18 岡本和樹"
